Commit message: AAA

File: urdf/robot.xacro (robot description, xacro)
@@ -27,5 +27,6 @@
     <inertial>
       <mass value="5.0"/>
-      <inertia ixx="0.1" ixy="0" ixz="0" iyy="0.1" iyz="0" izz="0.1"/>
+      <inertia ixx="0.043" ixy="0.0" ixz="0.0"
+              iyy="0.058" iyz="0.0" izz="0.043"/>
     </inertial>
   </link>
@@ -47,5 +48,6 @@
     <inertial>
       <mass value="0.5"/>
-      <inertia ixx="0.001" ixy="0.0" ixz="0.0" iyy="0.001" iyz="0.0" izz="0.001"/>
+      <inertia ixx="0.0001" ixy="0.0" ixz="0.0"
+              iyy="0.00128" iyz="0.0" izz="0.0001"/>
     </inertial>
   </link>
