Commit message: ab4
	修改：     CMakeLists.txt
	重命名：   build/.cmake/api/v1/reply/cache-v2-f2cd047c78adec7befd2.json -> build/.cmake/api/v1/reply/cache-v2-92993b4bcc411e3e6839.json
	重命名：   build/.cmake/api/v1/reply/codemodel-v2-0addace65dbfe8e3b7ed.json -> build/.cmake/api/v1/reply/codemodel-v2-c148a1aae10e21aee95e.json
	重命名：   build/.cmake/api/v1/reply/directory-.-Debug-d0ed23f2d20bac67032d.json -> build/.cmake/api/v1/reply/directory-.-Debug-c55478abdba0aefa62c4.json
	重命名：   build/.cmake/api/v1/reply/index-2025-06-12T11-03-56-0362.json -> build/.cmake/api/v1/reply/index-2025-06-13T13-43-02-0077.json
	重命名：   build/.cmake/api/v1/reply/target-controller-Debug-ab4014b06e0f7a204c1a.json -> build/.cmake/api/v1/reply/target-controller-Debug-ff8f28c16a25708b5469.json
	重命名：   build/.cmake/api/v1/reply/target-depth_processor-Debug-f1e135fc874ed3c50f97.json -> build/.cmake/api/v1/reply/target-depth_processor-Debug-d5016d7c3920bbcc0a45.json
	重命名：   build/.cmake/api/v1/reply/target-image_processor-Debug-920e3228ecd3b584a985.json -> build/.cmake/api/v1/reply/target-image_processor-Debug-7aacff5e3d8d02bcfa68.json
	重命名：   build/.cmake/api/v1/reply/target-uninstall-Debug-4003e0c7d87cd535b278.json -> build/.cmake/api/v1/reply/target-uninstall-Debug-d4bb04ce8124acd12a59.json
	重命名：   build/.cmake/api/v1/reply/target-vision_tracking_uninstall-Debug-47e96a8fd2041091085f.json -> build/.cmake/api/v1/reply/target-vision_tracking_uninstall-Debug-7d48deb4ec88f077ed8c.json
	修改：     build/CMakeCache.txt
	修改：     build/Testing/20250613-1000/Test.xml
	修改：     build/Testing/Temporary/LastTest_20250613-1000.log
	修改：     launch/simulation.launch.py
	修改：     rviz/tracking.rviz
	新文件：   urdf/robot.urdf
	修改：     urdf/robot.xacro

File: urdf/robot.urdf (robot description, URDF)
Before this commit: robot vision_tracking_robot, 5 links, 4 joints
Links:
- added link dummy_root_link, mass 0.001
- link base_link: geometry collision box size=0.4 0.3 0.15; visual box size=0.4 0.3 0.15
- link left_wheel: geometry collision cylinder length=0.04 radius=0.08; visual cylinder length=0.04 radius=0.08
- link right_wheel: geometry collision cylinder length=0.04 radius=0.08; visual cylinder length=0.04 radius=0.08
Joints:
- added joint dummy_root_to_base: type fixed, parent dummy_root_link, child base_link, origin xyz=0 0 0 rpy=0 0 0
- joint camera_joint: origin xyz=${camera_x_offset} 0.0 ${camera_z_offset} rpy=0 0 0 -> xyz=0.2 0.0 0.1 rpy=0 0 0
- joint caster_joint: origin xyz=${base_length/2} 0.0 -${base_height/2 + 0.01} -> xyz=0.2 0.0 -0.085 rpy=0 0 0
- joint left_wheel_joint: origin xyz=0.0 ${wheel_y_offset} -${base_height/2} -> xyz=0.0 0.15 -0.05 rpy=0 0 0
- joint right_wheel_joint: origin xyz=0.0 -${wheel_y_offset} -${base_height/2} -> xyz=0.0 -0.15 -0.05 rpy=0 0 0

Commit message: 重命名：   build/.cmake/api/v1/reply/cache-v2-92993b4bcc411e3e6839.json -> build/.cmake/api/v1/reply/cache-v2-efca0d14eb042fb589aa.json 	重命名：   build/.cmake/api/v1/reply/index-2025-06-13T13-43-02-0077.json -> build/.cmake/api/v1/reply/index-2025-06-14T11-51-09-0910.json 	修改：     build/CMakeCache.txt 	新文件：   build/Testing/20250614-1151/Test.xml 	修改：     build/Testing/TAG 	新文件：   build/Testing/Temporary/LastTest_20250614-1151.log 	修改：     urdf/robot.urdf 	修改：     worlds/empty.world

File: urdf/robot.urdf (robot description, URDF)
Before this commit: robot vision_tracking_robot, 6 links, 5 joints
Joints:
- joint camera_joint: origin xyz=0.2 0.0 0.1 rpy=0 0 0 -> xyz=0.2 0.0 0.2 rpy=0 0 0
- joint left_wheel_joint: origin xyz=0.0 0.15 -0.05 rpy=0 0 0 -> xyz=0.0 0.15 0.05 rpy=0 0 0

Commit message: 重命名：   build/.cmake/api/v1/reply/cache-v2-efca0d14eb042fb589aa.json -> build/.cmake/api/v1/reply/cache-v2-d248231d399cac75c7b2.json 	重命名：   build/.cmake/api/v1/reply/index-2025-06-14T11-51-09-0910.json -> build/.cmake/api/v1/reply/index-2025-06-14T12-44-11-0586.json 	修改：     build/CMakeCache.txt 	修改：     build/Testing/20250614-1151/Test.xml 	修改：     build/Testing/Temporary/LastTest_20250614-1151.log 	修改：     launch/simulation.launch.py 	修改：     rviz/tracking.rviz 	修改：     urdf/robot.urdf 	修改：     urdf/robot.xacro 	修改：     worlds/empty.world     修复世界问题，重写机器人urdf文件

File: urdf/robot.urdf (robot description, URDF)
Before this commit: robot vision_tracking_robot, 6 links, 5 joints
Links:
- removed link caster_wheel
- removed link dummy_root_link
- removed link left_wheel
- removed link right_wheel
- added link camera_base; visual box size=0.06 0.06 0.02
- added link camera_lens; visual cylinder length=0.01 radius=0.03
- added link camera_support; visual cylinder length=0.06 radius=0.01
- added link cockpit; visual box size=0.2 0.15 0.1
- added link wheel_fl, mass 0.5; collision cylinder length=0.02 radius=0.05; visual cylinder length=0.02 radius=0.05
- added link wheel_fr, mass 0.5; collision cylinder length=0.02 radius=0.05; visual cylinder length=0.02 radius=0.05
- added link wheel_rl, mass 0.5; collision cylinder length=0.02 radius=0.05; visual cylinder length=0.02 radius=0.05
- added link wheel_rr, mass 0.5; collision cylinder length=0.02 radius=0.05; visual cylinder length=0.02 radius=0.05
- link base_link: geometry collision box size=0.4 0.2 0.1; visual box size=0.4 0.2 0.1
- link camera_link: mass 0.1 -> None; geometry visual box size=0.09 0.07 0.07
Joints:
- removed joint camera_joint
- removed joint caster_joint
- removed joint dummy_root_to_base
- removed joint left_wheel_joint
- removed joint right_wheel_joint
- added joint joint_camera: type fixed, parent camera_support, child camera_link, origin xyz=0.045 0 0 rpy=0 0 0
- added joint joint_camera_base: type fixed, parent base_link, child camera_base, origin xyz=0.1 0 0.04 rpy=0 0 0
- added joint joint_camera_lens: type fixed, parent camera_link, child camera_lens, origin xyz=0.045 0 0 rpy=0 1.5708 0
- added joint joint_camera_support: type fixed, parent camera_base, child camera_support, origin xyz=0 0 0.04 rpy=0 0 0
- added joint joint_cockpit: type fixed, parent base_link, child cockpit, origin xyz=0 0 0.1 rpy=0 0 0
- added joint joint_wheel_fl: type continuous, parent base_link, child wheel_fl, origin xyz=0.15 0.1 -0.05 rpy=1.5708 0 0, axis 0 0 1
- added joint joint_wheel_fr: type continuous, parent base_link, child wheel_fr, origin xyz=0.15 -0.1 -0.05 rpy=1.5708 0 0, axis 0 0 1
- added joint joint_wheel_rl: type continuous, parent base_link, child wheel_rl, origin xyz=-0.15 0.1 -0.05 rpy=1.5708 0 0, axis 0 0 1
- added joint joint_wheel_rr: type continuous, parent base_link, child wheel_rr, origin xyz=-0.15 -0.1 -0.05 rpy=1.5708 0 0, axis 0 0 1

File: urdf/robot.xacro (robot description, xacro)
@@ -2,12 +2,14 @@
 <robot name="vision_tracking_robot" xmlns:xacro="http://www.ros.org/wiki/xacro">
   <!-- 基础参数 -->
-  <xacro:property name="base_length" value="0.4" />
-  <xacro:property name="base_width" value="0.3" />
-  <xacro:property name="base_height" value="0.15" />
-  <xacro:property name="wheel_radius" value="0.08" />
-  <xacro:property name="wheel_width" value="0.04" />
-  <xacro:property name="wheel_y_offset" value="0.15" />
-  <xacro:property name="camera_x_offset" value="0.2" />
-  <xacro:property name="camera_z_offset" value="0.1" />
+  <xacro:property name="base_length" value="0.4" />       <!-- 底盘长度 -->
+  <xacro:property name="base_width" value="0.3" />        <!-- 底盘宽度 -->
+  <xacro:property name="base_height" value="0.15" />      <!-- 底盘高度 -->
+  <xacro:property name="wheel_radius" value="0.08" />     <!-- 轮子半径 -->
+  <xacro:property name="wheel_width" value="0.04" />      <!-- 轮子宽度（轴向长度） -->
+  <xacro:property name="wheel_y_offset" value="0.07" />   <!-- 轮子y方向偏移（调整为底盘宽度的一半减去轮子半径） -->
+  <xacro:property name="camera_x_offset" value="0.2" />   <!-- 摄像头x方向偏移 -->
+  <xacro:property name="camera_z_offset" value="0.1" />   <!-- 摄像头z方向高度 -->
+  <xacro:property name="caster_radius" value="0.03" />    <!-- 支撑轮半径 -->
+  <xacro:property name="caster_x_offset" value="${base_length/2 - caster_radius}" />  <!-- 支撑轮x方向位置（确保在底盘范围内） -->
   <!-- 机器人底盘 -->
   <link name="base_link">
@@ -27,5 +29,6 @@
     <inertial>
       <mass value="5.0"/>
-      <inertia ixx="0.1" ixy="0.0" ixz="0.0" iyy="0.1" iyz="0.0" izz="0.1"/>
+      <inertia ixx="0.043" ixy="0.0" ixz="0.0"
+              iyy="0.058" iyz="0.0" izz="0.043"/>
     </inertial>
   </link>
@@ -36,6 +39,4 @@
         <cylinder radius="${wheel_radius}" length="${wheel_width}"/>
       </geometry>
-      <!-- 关键修改：添加自身旋转 -->
-      <origin rpy="1.5708 0 0" xyz="0 0 0"/>
       <material name="black">
         <color rgba="0.1 0.1 0.1 1.0"/>
@@ -46,10 +47,9 @@
         <cylinder radius="${wheel_radius}" length="${wheel_width}"/>
       </geometry>
-      <!-- 关键修改：添加自身旋转 -->
-      <origin rpy="1.5708 0 0" xyz="0 0 0"/>
     </collision>
     <inertial>
       <mass value="0.5"/>
-      <inertia ixx="0.001" ixy="0.0" ixz="0.0" iyy="0.001" iyz="0.0" izz="0.001"/>
+      <inertia ixx="0.0001" ixy="0.0" ixz="0.0"
+              iyy="0.00128" iyz="0.0" izz="0.0001"/>
     </inertial>
   </link>
@@ -57,6 +57,6 @@
     <parent link="base_link"/>
     <child link="left_wheel"/>
-    <!-- 关键修改：移除rpy旋转 -->
-    <origin xyz="0.0 ${wheel_y_offset} -${base_height/2}"/>
+    <!-- 调整y偏移量为0.07（底盘半宽0.15 - 轮子半径0.08 = 0.07），确保轮子在底盘范围内 -->
+    <origin xyz="0.0 ${wheel_y_offset} -${base_height/2}" rpy="0 1.5708 0"/>
     <axis xyz="0 1 0"/>
   </joint>
@@ -67,6 +67,4 @@
         <cylinder radius="${wheel_radius}" length="${wheel_width}"/>
       </geometry>
-      <!-- 关键修改：添加自身旋转 -->
-      <origin rpy="1.5708 0 0" xyz="0 0 0"/>
       <material name="black">
         <color rgba="0.1 0.1 0.1 1.0"/>
@@ -77,6 +75,4 @@
         <cylinder radius="${wheel_radius}" length="${wheel_width}"/>
       </geometry>
-      <!-- 关键修改：添加自身旋转 -->
-      <origin rpy="1.5708 0 0" xyz="0 0 0"/>
     </collision>
     <inertial>
@@ -88,13 +84,13 @@
     <parent link="base_link"/>
     <child link="right_wheel"/>
-    <!-- 关键修改：移除rpy旋转 -->
-    <origin xyz="0.0 -${wheel_y_offset} -${base_height/2}"/>
+    <!-- 调整y偏移量同上 -->
+    <origin xyz="0.0 -${wheel_y_offset} -${base_height/2}" rpy="0 1.5708 0"/>
     <axis xyz="0 1 0"/>
   </joint>
-  <!-- 前支撑轮 -->
+  <!-- 前支撑轮（调整为在底盘x范围内） -->
   <link name="caster_wheel">
     <visual>
       <geometry>
-        <sphere radius="0.03"/>
+        <sphere radius="${caster_radius}"/>
       </geometry>
       <material name="gray">
@@ -104,5 +100,5 @@
     <collision>
       <geometry>
-        <sphere radius="0.03"/>
+        <sphere radius="${caster_radius}"/>
       </geometry>
     </collision>
@@ -114,7 +110,6 @@
   <joint name="caster_joint" type="fixed">
     <parent link="base_link"/>
-    <child link="caster_wheel"/>
-    <!-- 优化：提高支撑轮高度 -->
-    <origin xyz="${base_length/2} 0.0 -${base_height/2 + 0.01}"/>
+    <!-- 支撑轮x坐标调整为底盘半长减去支撑轮半径，确保在底盘范围内 -->
+    <origin xyz="${caster_x_offset} 0.0 -${base_height/2}"/>
   </joint>
   <!-- 摄像头 -->
@@ -151,6 +146,6 @@
       <left_joint>left_wheel_joint</left_joint>
       <right_joint>right_wheel_joint</right_joint>
-      <wheel_separation>${2 * wheel_y_offset}</wheel_separation>
-      <wheel_diameter>${2 * wheel_radius}</wheel_diameter>
+      <wheel_separation>${2 * wheel_y_offset}</wheel_separation>  <!-- 轮距=2*轮子y偏移 -->
+      <wheel_diameter>${2 * wheel_radius}</wheel_diameter>       <!-- 轮径=2*轮子半径 -->
       <command_topic>cmd_vel</command_topic>
       <odometry_topic>odom</odometry_topic>
@@ -166,6 +161,5 @@
       <update_rate>30.0</update_rate>
       <camera name="camera">
-        <!-- 优化：扩大视野至80度 -->
-        <horizontal_fov>1.39626</horizontal_fov>
+        <horizontal_fov>1.0472</horizontal_fov> <!-- 60 degrees -->
         <image>
           <width>640</width>

Commit message: 最新版本。只差跟踪了

File: urdf/robot.urdf (robot description, URDF)
Before this commit: robot minimal_robot, 10 links, 9 joints
Links:
- link camera_base: mass None -> 0.1; geometry collision box size=0.06 0.06 0.02; visual box size=0.06 0.06 0.02
- link camera_lens: mass None -> 0.05; geometry collision cylinder length=0.01 radius=0.03; visual cylinder length=0.01 radius=0.03
- link camera_link: mass None -> 0.2; geometry collision box size=0.09 0.07 0.07; visual box size=0.09 0.07 0.07
- link camera_support: mass None -> 0.05; geometry collision cylinder length=0.06 radius=0.01; visual cylinder length=0.06 radius=0.01
